Commit message: changing continuous joints to revolute

File: kortex_description/arms/gen3/7dof/urdf/gen3.urdf (robot description, URDF)
Before this commit: robot gen3, 10 links, 9 joints
Joints:
- joint joint_1: limit effort=39 velocity=1.3963 -> lower=-20.0 upper=20.0 effort=39 velocity=1.3963; type continuous -> revolute
- joint joint_3: limit effort=39 velocity=1.3963 -> lower=-20.0 upper=20.0 effort=39 velocity=1.3963; type continuous -> revolute
- joint joint_5: limit effort=9 velocity=1.2218 -> lower=-20.0 upper=20.0 effort=9 velocity=1.2218; type continuous -> revolute
- joint joint_7: limit effort=9 velocity=1.2218 -> lower=-20.0 upper=20.0 effort=9 velocity=1.2218; type continuous -> revolute

File: kortex_description/arms/gen3/7dof/urdf/gen3_macro.xacro (robot description, xacro)
@@ -62,5 +62,5 @@
     <joint
       name="${prefix}joint_1"
-      type="continuous">
+      type="revolute">
       <origin xyz="0 0 0.15643" rpy="3.1416 2.7629E-18 -4.9305E-36" />
       <parent
@@ -72,5 +72,5 @@
       <limit
         effort="39"
-        velocity="1.3963" />
+        velocity="1.3963"  upper="20" lower="-20"/>
     </joint>
     <link name="${prefix}half_arm_1_link">
@@ -132,5 +132,5 @@
     <joint
       name="${prefix}joint_3"
-      type="continuous">
+      type="revolute">
       <origin xyz="0 -0.21038 -0.006375" rpy="-1.5708 1.2326E-32 -2.9122E-16" />
       <parent
@@ -142,5 +142,5 @@
       <limit
         effort="39"
-        velocity="1.3963" />
+        velocity="1.3963"  upper="20" lower="-20"/>
     </joint>
     <link name="${prefix}forearm_link">
@@ -202,5 +202,5 @@
     <joint
       name="${prefix}joint_5"
-      type="continuous">
+      type="revolute">
       <origin xyz="0 -0.20843 -0.006375" rpy="-1.5708 2.2204E-16 -6.373E-17" />
       <parent
@@ -212,5 +212,5 @@
       <limit
         effort="9"
-        velocity="1.2218" />
+        velocity="1.2218" upper="20" lower="-20"/>
     </joint>
     <link name="${prefix}spherical_wrist_2_link">
@@ -298,5 +298,5 @@
     <joint
       name="${prefix}joint_7"
-      type="continuous">
+      type="revolute">
       <origin xyz="0 -0.10593 -0.00017505" rpy="-1.5708 -5.5511E-17 9.6396E-17" />
       <parent
@@ -308,5 +308,5 @@
       <limit
         effort="9"
-        velocity="1.2218" />
+        velocity="1.2218"  upper="20" lower="-20"/>
     </joint>
     <link name="${prefix}end_effector_link" />
