Commit message: adding dummy link with inertia for the base

File: kortex_description/arms/gen3/7dof/urdf/gen3_macro.xacro (robot description, xacro)
@@ -5,9 +5,9 @@
   <xacro:macro name="load_arm" params="parent:='' dof vision prefix *origin">
       <link name="${prefix}base_link">
-        <inertial>
+        <!-- <inertial>
           <origin xyz="-0.000648 -0.000166 0.084487" rpy="0 0 0" />
           <mass value="1.697" />
           <inertia ixx="0.004622" ixy="9E-06" ixz="6E-05" iyy="0.004495" iyz="9E-06" izz="0.002079" />
-        </inertial>
+        </inertial> -->
         <visual>
           <origin xyz="0 0 0" rpy="0 0 0" />
@@ -26,4 +26,16 @@
         </collision>
     </link>
+    <link name="${prefix}base_link_dummy">
+      <inertial>
+        <origin rpy="0 0 0" xyz="-0.000648 -0.000166 0.084487"/>
+        <mass value="1.697"/>
+        <inertia ixx="0.004622" ixy="9E-06" ixz="6E-05" iyy="0.004495" iyz="9E-06" izz="0.002079"/>
+      </inertial>
+    </link>
+    <joint name="${prefix}base_dummy_joint" type="fixed">
+      <origin rpy="0.0 0.0 0.0" xyz="0 0 0"/>
+      <parent link="${prefix}base_link"/>
+      <child link="${prefix}base_link_dummy"/>
+    </joint>
     <link name="${prefix}shoulder_link">
       <inertial>

Commit message: working admittance mpc controller -- need some tuning

File: kortex_description/arms/gen3/7dof/urdf/gen3_macro.xacro (robot description, xacro)
@@ -296,5 +296,5 @@
     </link>
     </xacro:unless>
-    <joint
+      <joint
       name="${prefix}joint_7"
       type="revolute">
@@ -343,3 +343,17 @@
     </xacro:if>
   </xacro:macro>
+  <!--      Interconnect link : where the imu is placed-->
+      <link name="${prefix}interconnect_link" />
+      <joint name="${prefix}interconnect_joint" type="fixed">
+        <parent link="${prefix}end_effector_link"/>
+        <child link="${prefix}interconnect_link"/>
+        <origin xyz="0 0 0" rpy="3.14159 0 0.0" />
+      </joint>
+<!--      FT Sensor link : aligned with the interconnect link -->
+      <link name="ft_sensor0" />
+      <joint name="${prefix}ft_sensor_joint" type="fixed">
+        <parent link="${prefix}end_effector_link"/>
+        <child link="ft_sensor0"/>
+        <origin xyz="0 0 0" rpy="0 0 -1.57079" />
+      </joint>
 </robot>

Commit message: last changes before switching to local package

File: kortex_description/arms/gen3/7dof/urdf/gen3_macro.xacro (robot description, xacro)
@@ -351,5 +351,15 @@
       </joint>
 <!--      FT Sensor link : aligned with the interconnect link -->
-      <link name="ft_sensor0" />
+      <link name="ft_sensor0">
+        <visual>
+          <origin xyz="0 0 0.03" rpy="0 0 3.14" />
+          <geometry>
+            <mesh filename="package://kortex_description/arms/gen3/${dof}dof/meshes/bota_sensor.stl" scale="0.001 0.001 0.001"/>
+          </geometry>
+          <material name="">
+            <color rgba="0.75294 0.75294 0.75294 1" />
+          </material>
+        </visual>
+      </link>
       <joint name="${prefix}ft_sensor_joint" type="fixed">
         <parent link="${prefix}end_effector_link"/>

File: kortex_description/robots/gen3_robotiq_2f_85.xacro (robot description, xacro)
@@ -8,5 +8,6 @@
     <xacro:arg name="sim" default="false" />
     <xacro:arg name="prefix" default="" />
+    <xacro:arg name="tool_frame_offset" default="0.12"/>
     <xacro:include filename="$(find kortex_description)/robots/kortex_robot.xacro" />
-    <xacro:load_robot arm="$(arg arm)" gripper="$(arg gripper)" dof="$(arg dof)" vision="$(arg vision)" sim="$(arg sim)" prefix="$(arg prefix)" />
+    <xacro:load_robot arm="$(arg arm)" gripper="$(arg gripper)" dof="$(arg dof)" vision="$(arg vision)" sim="$(arg sim)" prefix="$(arg prefix)" tool_frame_offset="$(arg tool_frame_offset)"/>
 </robot>
