Commit message: lowlevel gripper integration

File: kortex_move_it_config/gen3_robotiq_2f_85_move_it_config/config/7dof/gen3_robotiq_2f_85.srdf.xacro (robot description, xacro)
@@ -37,5 +37,5 @@
     <!--GROUP STATES: Purpose: Define a named state for a particular group, in terms of joint values. This is useful to define states like 'folded arms'-->
     <group_state name="home" group="arm">
-        <joint name="$(arg prefix)joint_1" value="0" />
+        <joint name="$(arg prefix)joint_1" value="-1.57" />
         <joint name="$(arg prefix)joint_2" value="0.26" />
         <joint name="$(arg prefix)joint_3" value="3.14" />
