Commit message: same tool frame  with and without gripper

File: kortex_description/robots/kortex_robot.xacro (robot description, xacro)
@@ -38,5 +38,5 @@
             <link name="${prefix}tool_frame"/>
             <joint name="${prefix}tool_frame_joint" type="fixed">
-                <origin xyz="0 0 0" rpy="0 0 0" />
+                <origin xyz="0 0 0.12" rpy="0 0 0" />
                 <parent link="${prefix}${last_arm_link}" />
                 <child link="${prefix}tool_frame" />
