Commit message: specifying tool offset frame

File: kortex_description/robots/gen3.xacro (robot description, xacro)
@@ -8,4 +8,6 @@
     <xacro:arg name="sim" default="false" />
     <xacro:arg name="prefix" default="" />
+    <xacro:arg name="tool_frame_offset" default="0.12"/>
+    <xacro:property name="tool_frame_offset" default="$(arg tool_frame_offset)"/>
     <xacro:include filename="$(find kortex_description)/robots/kortex_robot.xacro" />
     <xacro:load_robot arm="$(arg arm)" gripper="$(arg gripper)" dof="$(arg dof)" vision="$(arg vision)" sim="$(arg sim)" prefix="$(arg prefix)" />

File: kortex_description/robots/kortex_robot.xacro (robot description, xacro)
@@ -38,5 +38,5 @@
             <link name="${prefix}tool_frame"/>
             <joint name="${prefix}tool_frame_joint" type="fixed">
-                <origin xyz="0 0 0.12" rpy="0 0 0" />
+                <origin xyz="0 0 ${tool_frame_offset}" rpy="0 0 0" />
                 <parent link="${prefix}${last_arm_link}" />
                 <child link="${prefix}tool_frame" />

Commit message: tool_offset param

File: kortex_description/robots/gen3.xacro (robot description, xacro)
@@ -9,6 +9,5 @@
     <xacro:arg name="prefix" default="" />
     <xacro:arg name="tool_frame_offset" default="0.12"/>
-    <xacro:property name="tool_frame_offset" default="$(arg tool_frame_offset)"/>
     <xacro:include filename="$(find kortex_description)/robots/kortex_robot.xacro" />
-    <xacro:load_robot arm="$(arg arm)" gripper="$(arg gripper)" dof="$(arg dof)" vision="$(arg vision)" sim="$(arg sim)" prefix="$(arg prefix)" />
+    <xacro:load_robot arm="$(arg arm)" gripper="$(arg gripper)" dof="$(arg dof)" vision="$(arg vision)" sim="$(arg sim)" prefix="$(arg prefix)" tool_frame_offset="$(arg tool_frame_offset)"/>
 </robot>

File: kortex_description/robots/kortex_robot.xacro (robot description, xacro)
@@ -1,5 +1,5 @@
 <?xml version="1.0"?>
 <robot xmlns:xacro="http://ros.org/wiki/xacro">
-    <xacro:macro name="load_robot" params="arm gripper dof vision sim prefix">
+    <xacro:macro name="load_robot" params="arm gripper dof vision sim prefix tool_frame_offset">
         <!-- Files to include -->
         <xacro:include filename="$(find kortex_description)/arms/${arm}/${dof}dof/urdf/${arm}_macro.xacro" />
