Commit message: terminating the kinematic chain at the end effector link to avoid discrepancies when the tool frame is moved for different payloads

File: kortex_move_it_config/gen3_move_it_config/config/7dof/gen3.srdf.xacro (robot description, xacro)
@@ -20,5 +20,5 @@
         <joint name="$(arg prefix)joint_7" />
         <joint name="$(arg prefix)end_effector" />
-        <joint name="$(arg prefix)tool_frame_joint" />
+        <!-- <joint name="$(arg prefix)tool_frame_joint" /> -->
     </group>
     <!--GROUP STATES: Purpose: Define a named state for a particular group, in terms of joint values. This is useful to define states like 'folded arms'-->
